Commit message: 1

File: src/spider_description/urdf/spider.urdf (robot description, URDF)
Before this commit: robot spider, 20 links, 19 joints
Joints:
- joint left-front-coxae: axis 0 0 0 -> 0 1 0

Commit message: final

File: src/spider_description/urdf/spider.urdf (robot description, URDF)
Before this commit: robot spider, 20 links, 19 joints
Links:
- added link head2, mass 1; collision box size=0.2 0.2 0.2; visual box size=0.2 0.2 0.2
- added link tetris; visual box size=2 4 0.347
Joints:
- added joint modeyong: type continuous, parent body, child tetris, origin xyz=0 0 0 rpy=0 0 0, axis 1 0 0, limit lower=0 upper=0 effort=0 velocity=0
- added joint neck2: type fixed, parent body, child head2, origin xyz=0 0 0 rpy=0 0 0, axis 1 0 0, limit lower=0 upper=0 effort=0 velocity=0

File: src/spider_description/urdf/step1.urdf (robot description, URDF)
Before this commit: robot spider, 20 links, 19 joints
Links:
- added link head2, mass 1; collision box size=0.2 0.2 0.2; visual box size=0.2 0.2 0.2
Joints:
- added joint neck2: type fixed, parent body, child head2, origin xyz=0 0 0 rpy=0 0 0, axis 1 0 0, limit lower=0 upper=0 effort=0 velocity=0
- joint left-back-ankle: axis 0 0 0 -> 1 0 0
- joint left-back-coxae: axis 0 0 0 -> 1 0 0
- joint left-back-knee: axis 0 0 0 -> 1 0 0
- joint left-front-ankle: axis 0 0 0 -> 1 0 0
- joint left-front-coxae: axis 0 0 0 -> 1 0 0
- joint left-front-knee: axis 0 0 0 -> 1 0 0
- joint left-middle-ankle: axis 0 0 0 -> 1 0 0
- joint left-middle-coxae: axis 0 0 0 -> 1 0 0
- joint left-middle-knee: axis 0 0 0 -> 1 0 0
- joint neck: axis 0 0 0 -> 1 0 0
- joint right-back-ankle: axis 0 0 0 -> 1 0 0
- joint right-back-coxae: axis 0 0 0 -> 1 0 0
- joint right-back-knee: axis 0 0 0 -> 1 0 0
- joint right-front-ankle: axis 0 0 0 -> 1 0 0
- joint right-front-coxae: axis 0 0 0 -> 1 0 0
- joint right-front-knee: axis 0 0 0 -> 1 0 0
- joint right-middle-ankle: axis 0 0 0 -> 1 0 0
- joint right-middle-coxae: axis 0 0 0 -> 1 0 0
- joint right-middle-knee: axis 0 0 0 -> 1 0 0

File: src/spider_description/urdf/tai135.urdf (robot description, URDF)
Before this commit: robot spider, 20 links, 19 joints
Links:
- added link head2, mass 1; collision box size=0.2 0.2 0.2; visual box size=0.2 0.2 0.2
Joints:
- added joint neck2: type fixed, parent body, child head2, origin xyz=0 0 0 rpy=0 0 0, axis 1 0 0, limit lower=0 upper=0 effort=0 velocity=0

File: src/spider_description/urdf/tai246.urdf (robot description, URDF)
Before this commit: robot spider, 20 links, 19 joints
Links:
- added link head2, mass 1; collision box size=0.2 0.2 0.2; visual box size=0.2 0.2 0.2
Joints:
- added joint neck2: type fixed, parent body, child head2, origin xyz=0 0 0 rpy=0 0 0, axis 1 0 0, limit lower=0 upper=0 effort=0 velocity=0

File: src/spider_description/urdf/tetris1.urdf (robot description, URDF)
Before this commit: robot spider, 20 links, 19 joints
Links:
- added link head2, mass 1; collision box size=0.2 0.2 0.2; visual box size=0.2 0.2 0.2
- added link tetris; visual box size=2 4 0.347
Joints:
- added joint modeyong: type continuous, parent body, child tetris, origin xyz=0 0 0 rpy=0 0 0, axis 1 0 0, limit lower=0 upper=0 effort=0 velocity=0
- added joint neck2: type fixed, parent body, child head2, origin xyz=0 0 0 rpy=0 0 0, axis 1 0 0, limit lower=0 upper=0 effort=0 velocity=0
- joint left-back-ankle: axis 0 0 0 -> 1 0 0
- joint left-back-coxae: axis 0 0 0 -> 1 0 0
- joint left-back-knee: axis 0 0 0 -> 1 0 0
- joint left-front-ankle: axis 0 0 0 -> 1 0 0
- joint left-front-coxae: axis 0 0 0 -> 1 0 0
- joint left-front-knee: axis 0 0 0 -> 1 0 0
- joint left-middle-ankle: axis 0 0 0 -> 1 0 0
- joint left-middle-coxae: axis 0 0 0 -> 1 0 0
- joint left-middle-knee: axis 0 0 0 -> 1 0 0
- joint neck: axis 0 0 0 -> 1 0 0
- joint right-back-ankle: axis 0 0 0 -> 1 0 0
- joint right-back-coxae: axis 0 0 0 -> 1 0 0
- joint right-back-knee: axis 0 0 0 -> 1 0 0
- joint right-front-ankle: axis 0 0 0 -> 1 0 0
- joint right-front-coxae: axis 0 0 0 -> 1 0 0
- joint right-front-knee: axis 0 0 0 -> 1 0 0
- joint right-middle-ankle: axis 0 0 0 -> 1 0 0
- joint right-middle-coxae: axis 0 0 0 -> 1 0 0
- joint right-middle-knee: axis 0 0 0 -> 1 0 0
